File: schmatic/schmatic.kicad_sch (KiCad schematic)
At the start: 10 parts, among them J1 RFIO-RC522, J2 RTC, U1 LCD-016N002L

Commit message: ready to demo
Connections:
- net +5V: no longer U1.5 (R/~{W})
- net GND: now also U1.5 (R/~{W})
Changed lines of the file:
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@@
-    (stroke (width 0) (type default))
-  )
-  (wire (pts (xy 105.41 114.3) (xy 105.41 101.6))
     (stroke (width 0) (type default))
   )
@@
   )
   (wire (pts (xy 104.14 86.36) (xy 104.14 90.17))
+    (stroke (width 0) (type default))
+  )
+  (wire (pts (xy 105.41 149.86) (xy 134.62 149.86))
     (stroke (width 0) (type default))
   )
@@
     (stroke (width 0) (type default))
   )
-  (wire (pts (xy 105.41 101.6) (xy 134.62 101.6))
-    (stroke (width 0) (type default))
-  )
   (wire (pts (xy 198.12 77.47) (xy 201.93 77.47))
     (stroke (width 0) (type default))
@@
     (stroke (width 0) (type default))
   )
+  (wire (pts (xy 105.41 114.3) (xy 105.41 149.86))
+    (stroke (width 0) (type default))
+  )
